File: hardware/zvire-vetrnik-power/zvire-vetrnik-power.kicad_pcb (KiCad board)
At the start: 2 copper layers, 158.8 x 99.1 mm, 132 parts, among them J1 12V IN, J10 AC frequency sense, J11 AVR-ISP-6, J12 ACS712_2, J13 ACS712, J2 ~SHORT, J3 UART, J4 ENABLE, J5 RELAYS, J6 DC IN, J7 PE, J8 CURRENT SENSOR, J9 AC OUT, M1 12V / 0,9A max, Q1 BCP56-16, Q10 IXFP90N20X3M, Q11 IXFP90N20X3M, Q12 IXFP90N20X3M, Q13 BC847, Q14 BC846, Q2 BC847, Q3 BC846, Q4 BC846, Q5 BC846, Q6 BC846, Q7 BC846, Q8 BC846, Q9 IXFP90N20X3M, SW1 AVR RESET, U1 LTV-847, U2 H11L1, U3 H11L1, U4 LTV-847, U5 LM393, U6 IR2104, U7 IR2104, U8 L78L05_TO92, U9 ATmega8-16PU, Y1 16MHz

Commit message: Vyrobena verze power PCB
Parts:
- removed Q11, Q12: IXFP90N20X3M, Package_TO_SOT_THT:TO-220F-3_Vertical
- removed Q13: BC847, Package_TO_SOT_SMD:SOT-23
- removed Q14: BC846, Package_TO_SOT_SMD:SOT-23
- removed the U9 at (201.9, 59.7)
- added J10: AC1, ondra:FS1536, F.Cu at (112.9, 58.2)
- added J15: AVR-ISP-6, Connector_IDC:IDC-Header_2x03_P2.54mm_Vertical, F.Cu at (156.2, 138.4)
- added J16: ACS712_2, Connector_Molex:Molex_KK-254_AE-6410-03A_1x03_P2.54mm_Vertical, F.Cu at (151.1, 116.8)
- added J17: ACS712, Connector_Molex:Molex_KK-254_AE-6410-03A_1x03_P2.54mm_Vertical, F.Cu at (151.1, 120.7)
- added JP1: Jumper, Resistor_SMD:R_1206_3216Metric_Pad1.30x1.75mm_HandSolder, B.Cu at (139.7, 129.5)
- added JP2: Jumper, Resistor_SMD:R_1206_3216Metric_Pad1.30x1.75mm_HandSolder, B.Cu at (189.2, 81.3)
- added NT1: Net-Tie_2, NetTie:NetTie-2_SMD_Pad2.0mm, B.Cu at (106.0, 120.7)
- added U10: LTV-817, Package_DIP:DIP-4_W7.62mm, F.Cu at (191.8, 68.6)
- added U12: ATmega8-16PU, Package_DIP:DIP-28_W7.62mm_Socket, F.Cu at (135.9, 113.0)
- added U6: LTV-847, Package_DIP:DIP-16_W7.62mm, F.Cu at (176.5, 115.6)
- added U7: LM393, Package_SO:SOIC-8_3.9x4.9mm_P1.27mm, B.Cu at (122.6, 90.2)
- C10, C13, C16, C18, C19, C27, C28, C29, C3, C30, C31, C32, C4, C5, D5, D6, Q1, Q2, Q3, Q4, Q5, Q6, Q7, Q8, R1, R10, R11, R12, R13, R14, R15, R16, R17, R18, R19, R2, R20, R21, R22, R24, R25, R26, R28, R29, R3, R30, R31, R32, R33, R34, R36, R37, R38, R39, R4, R41, R42, R43, R44, R45, R46, R47, R5, R6, R7, R8, R9: moved to B.Cu
- J11: value AVR-ISP-6 -> AC2; footprint Connector_IDC:IDC-Header_2x03_P2.54mm_Vertical -> ondra:FS1536
- J12: value ACS712_2 -> G #Q3; footprint Connector_Molex:Molex_KK-254_AE-6410-03A_1x03_P2.54mm_Vertical -> Connector_Molex:Molex_KK-254_AE-6410-02A_1x02_P2.54mm_Vertical
- J13: value ACS712 -> G #Q4; footprint Connector_Molex:Molex_KK-254_AE-6410-03A_1x03_P2.54mm_Vertical -> Connector_Molex:Molex_KK-254_AE-6410-02A_1x02_P2.54mm_Vertical
- J8: value CURRENT SENSOR -> G #Q1; footprint ondra:DG270-10.0-02P-14-00A -> Connector_Molex:Molex_KK-254_AE-6410-02A_1x02_P2.54mm_Vertical
- J9: value AC OUT -> G #Q2; footprint ondra:DG270-10.0-02P-14-00A -> Connector_Molex:Molex_KK-254_AE-6410-02A_1x02_P2.54mm_Vertical
- Q10: value IXFP90N20X3M -> BC846; footprint Package_TO_SOT_THT:TO-220F-3_Vertical -> Package_TO_SOT_SMD:SOT-23; moved to B.Cu
- Q9: value IXFP90N20X3M -> BC847; footprint Package_TO_SOT_THT:TO-220F-3_Vertical -> Package_TO_SOT_SMD:SOT-23; moved to B.Cu
- TH1: footprint Resistor_THT:R_Axial_DIN0204_L3.6mm_D1.6mm_P2.54mm_Vertical -> Connector_Molex:Molex_KK-254_AE-6410-02A_1x02_P2.54mm_Vertical
- U1: value LTV-847 -> LTV-817; footprint Package_DIP:DIP-16_W7.62mm -> Package_DIP:DIP-4_W7.62mm
- U11: renamed from U8; footprint Package_TO_SOT_THT:TO-92_Inline -> Package_TO_SOT_THT:TO-92L_HandSolder
- U2: value H11L1 -> LTV-817; footprint Package_DIP:DIP-6_W7.62mm_LongPads -> Package_DIP:DIP-4_W7.62mm
- U4: value LTV-847 -> H11L1; footprint Package_DIP:DIP-16_W7.62mm -> Package_DIP:DIP-6_W7.62mm_LongPads
- U5: value LM393 -> LTV-817; footprint Package_SO:SOIC-8_3.9x4.9mm_P1.27mm -> Package_DIP:DIP-4_W7.62mm
- U8: renamed from U6; moved to B.Cu
- U9: renamed from U7; moved to B.Cu
- Y1: footprint Crystal:Crystal_SMD_HC49-SD_HandSoldering -> Crystal:Crystal_HC49-U_Vertical; moved to F.Cu
- moved R25 228.7 mm to (123.2, 97.8), turned to 180 degrees
- moved R29 219.9 mm to (123.2, 95.2), turned to 180 degrees
- moved R28 213.9 mm to (106.7, 114.3), turned to 180 degrees
- moved R26 210.1 mm to (118.1, 95.2), turned to 180 degrees
- moved R27 207.8 mm to (111.8, 104.1), turned to 270 degrees
- moved R24 202.4 mm to (106.7, 116.8), turned to 180 degrees
- moved R32 201.3 mm to (147.3, 76.2), turned to 180 degrees
- moved Q8 198.9 mm to (127.0, 91.4)
- moved R31 195.2 mm to (147.3, 78.7), turned to 180 degrees
- moved R30 186.7 mm to (128.3, 95.2), turned to 180 degrees
- moved R23 180.3 mm to (115.6, 104.1), turned to 270 degrees
- moved R2 179.6 mm to (176.5, 144.5), turned to 90 degrees
- moved R44 171.0 mm to (133.3, 127.0), turned to 90 degrees
- moved R38 170.2 mm to (166.4, 77.5), turned to 180 degrees
- moved J1 169.3 mm to (114.3, 146.1), turned to 180 degrees
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- renumbered J10 to J14
Connections:
- C12 pad 2: GNDPWR -> Net-(C12-Pad2)
- C13 pad 2: GNDPWR -> Net-(C12-Pad2)
- C14 pad 2: /H-bridge/AC1 -> Net-(C14-Pad2)
- C15 pad 2: GNDPWR -> Net-(C15-Pad2)
- C16 pad 2: GNDPWR -> Net-(C15-Pad2)
- C3 pad 2: GND -> /GND_UART
- C7 pad 2: Net-(C7-Pad2) -> /H-bridge/DC-
- C8 pad 2: GNDPWR -> /H-bridge/DC-
- C9 pad 2: GNDPWR -> /H-bridge/DC-
- D1 pad 1: Net-(C7-Pad2) -> /H-bridge/DC-
- D3 pad 1: /H-bridge/AC2 -> Net-(D3-Pad1)
- D3 pad 2: /H-bridge/AC1 -> Net-(C14-Pad2)
- J1 pad 1: GND -> +12V
- J1 pad 2: +12V -> GND
- J11 pad 1: /AVR MCU/MISO -> Net-(D3-Pad1)
- J12 pad 1: +5P -> Net-(C15-Pad2)
- J12 pad 2: /AVR MCU/ADC2_ACS712_2 -> Net-(J12-Pad2)
- J13 pad 1: +5P -> GNDPWR
- J13 pad 2: /AVR MCU/ADC1_ACS712 -> Net-(J13-Pad2)
- J14 pad 1: Net-(D5-Pad2) -> Net-(J14-Pad1)
- J14 pad 2: Net-(J10-Pad2) -> Net-(D5-Pad2)
- J3 pad 4: GND -> Net-(J3-Pad4)
- J4 pad 1: GND -> /ENABLE
- J4 pad 2: /ENABLE -> GND
- J5 pad 1: +12V -> GND
- J5 pad 2: /REL4 -> /REL1
- J5 pad 3: /REL3 -> /REL2
- J5 pad 4: /REL2 -> /REL3
- J5 pad 5: /REL1 -> /REL4
- J5 pad 6: GND -> +12V
- J6 pad 1: Net-(C7-Pad2) -> /H-bridge/DC-
- J8 pad 1: GNDPWR -> Net-(C12-Pad2)
- J8 pad 2: Net-(C7-Pad2) -> Net-(J8-Pad2)
- J9 pad 1: /H-bridge/AC1 -> GNDPWR
- J9 pad 2: /H-bridge/AC2 -> Net-(J9-Pad2)
- Q10 pad 2: /H-bridge/AC1 -> GNDPWR
- Q10 pad 3: GNDPWR -> /AVR MCU/SHORT
- Q9 pad 2: /H-bridge/DC+ -> GNDPWR
- Q9 pad 3: /H-bridge/AC1 -> /AVR MCU/RPM
- R24 pad 2: GNDPWR -> /H-bridge/DC-
- R28 pad 2: GNDPWR -> /H-bridge/DC-
- R33 pad 1: Net-(Q9-Pad1) -> Net-(J8-Pad2)
- R34 pad 1: Net-(Q10-Pad1) -> Net-(J9-Pad2)
- R35 pad 1: /H-bridge/AC2 -> Net-(D3-Pad1)
- R36 pad 2: Net-(Q11-Pad1) -> Net-(J12-Pad2)
- R37 pad 2: Net-(Q12-Pad1) -> Net-(J13-Pad2)
- R40 pad 2: Net-(J10-Pad2) -> Net-(J14-Pad1)
- R42 pad 1: Net-(Q13-Pad1) -> Net-(Q9-Pad1)
- R43 pad 1: Net-(Q13-Pad1) -> Net-(Q9-Pad1)
- R46 pad 1: Net-(Q14-Pad1) -> Net-(Q10-Pad1)
- U1 pad 3: Net-(R8-Pad2) -> Net-(R4-Pad1)
- U1 pad 4: GNDPWR -> +12V
- U2 pad 1: +5P -> Net-(R8-Pad2)
- U2 pad 2: Net-(R9-Pad2) -> GNDPWR
- U2 pad 3: Net-(U2-Pad3) -> Net-(Q2-Pad1)
- U2 pad 4: /TX -> +12V
- U3 pad 1: Net-(R6-Pad2) -> +5P
- U3 pad 2: /RX -> Net-(R9-Pad2)
- U3 pad 4: /AVR MCU/RX -> /TX
- U3 pad 5: GNDPWR -> /GND_UART
- U3 pad 6: +5P -> /3V3_UART
- U4 pad 1: Net-(R11-Pad1) -> Net-(R6-Pad2)
- U4 pad 2: GNDPWR -> /RX
- U4 pad 3: Net-(R12-Pad1) -> Net-(U4-Pad3)
- U4 pad 4: GNDPWR -> /AVR MCU/RX
- U4 pad 5: Net-(R13-Pad1) -> GNDPWR
- U4 pad 6: GNDPWR -> +5P
- U5 pad 1: Net-(Q8-Pad1) -> Net-(R5-Pad1)
- U5 pad 2: Net-(R27-Pad2) -> GND
- U5 pad 3: Net-(R25-Pad2) -> GNDPWR
- U5 pad 4: GNDPWR -> /AVR MCU/~ENABLE
- U8 pad 6: /H-bridge/AC1 -> Net-(C12-Pad2)
- U9 pad 6: /H-bridge/AC2 -> Net-(C15-Pad2)
Routing:
- net +12V: track 0.00 -> 238.2 mm, vias 0 -> 2
- net GNDPWR: track 217.9 -> 443.8 mm, vias 0 -> 4
- net GND: track 0.00 -> 213.4 mm, vias 0 -> 12
- net /H-bridge/DC+: track 371.4 -> 161.9 mm
- net +5P: track 0.00 -> 200.4 mm, vias 0 -> 4
- net +12P: track 0.00 -> 163.1 mm, vias 0 -> 6
- net /AVR MCU/~SD: track 0.00 -> 130.6 mm, vias 0 -> 2
- net /H-bridge/DC-: track 0.00 -> 129.0 mm
- net Net-(C7-Pad2): track 127.1 -> 0.00 mm
- net /H-bridge/AC2: track 108.7 -> 0.00 mm
- net /H-bridge/IN1: track 0.00 -> 104.6 mm, vias 0 -> 2
- net /AVR MCU/~SHORT: track 0.00 -> 92.7 mm, vias 0 -> 2
- net /H-bridge/IN2: track 0.00 -> 92.0 mm, vias 0 -> 2
- net /AVR MCU/TX: track 0.00 -> 81.5 mm, vias 0 -> 4
- net Net-(Q2-Pad1): track 0.00 -> 80.9 mm, vias 0 -> 4
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- added copper zone on B.Cu, net Net-(M1-Pad2)
Other:
- board size 158.8 x 99.1 mm -> 124.5 x 99.1 mm
