File: hardware/zvire-vetrnik-power-supply/zvire-vetrnik-power-supply.kicad_pcb (KiCad board)
At the start: 2 copper layers, 80 x 21.6 mm, 21 parts, among them J1 Conn_01x02, J2 Conn_01x04, J3 Conn_01x04, J4 Conn_01x04, U1 LM2575-3.3BT, U2 LM7805_TO220

Commit message: [hardware] Update PCB designs
Other:
- board text added: "12V"
- board text added: "12V IN"
- board text added: "12V Isense --->"
- board text added: "3V3"
- board text added: "3V3 Isense --->"
- board text added: "5V"
- board text added: "5V Isense --->"
- board text added: "GND"
- board text added: "TODO: next time, plan heatsinks better"
