File: hardware/zvire-vetrnik-control/zvire-vetrnik-control.kicad_pcb (KiCad board)
At the start: 2 copper layers, 99.1 x 76.2 mm, 87 parts, among them J1 Conn_01x20_Male, J10 Conn_01x04, J11 Conn_01x03_Male, J12 Conn_02x04_Odd_Even, J13 Conn_02x04_Odd_Even, J14 Conn_02x04_Odd_Even, J15 Conn_01x04, J16 Conn_01x04, J17 Conn_01x04, J18 Conn_01x03, J19 Conn_01x04, J2 Conn_01x04, J20 Conn_01x04, J3 Conn_01x03, J4 Conn_02x04_Odd_Even, J5 Conn_02x04_Odd_Even, J6 Conn_02x04_Odd_Even, J7 Conn_01x20_Male, J8 Screw_Terminal_01x02, J9 Conn_01x03, Q1 BC857, Q2 BC847, Q3 BC847, Q4 BC847, Q5 BSS138, Q6 BSS138, Q7 BC847, Q8 BSS138, SW1 SW_Push, SW2 SW_Push, U1 LTV-817S, U2 YAAJ_WeAct_BlackPill_Part_Like, U3 MX25L8006EM1I-12G, U4 WIZ850io

Commit message: [hardware] Update PCB designs
Other:
- board text added: "TODO: next time, do NCC (non-copper clearing) around optocoupler"
Changed lines of the file:
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@@
   (general
     (thickness 1.6)
-    (drawings 56)
+    (drawings 57)
     (tracks 745)
     (zones 0)
@@
     )
   )
+  (gr_text "TODO: next time, do NCC (non-copper clearing) around optocoupler" (at 216.535 164.465) (layer Cmts.User)
+    (effects (font (size 1.5 1.5) (thickness 0.3)))
+  )
   (gr_text ".\n." (at 58.42 133.35) (layer F.SilkS)

Commit message: [hardware] Add notes to control PCB design
Other:
- board text added: "TODO why is H2 moved 1.27mm off its intended position?"
