File: hardware/vetrnik-current-sensor/vetrnik-current-sensor.kicad_pcb (KiCad board)
At the start: 2 copper layers, 50.8 x 59.7 mm, 8 parts, among them J1 DG270-10.0-02P, J2 Conn_01x03, U1 ACS770xCB-050U-PFF

Commit message: Migrate KiCAD projects to KiCAD 7.0
Other:
- net class Default removed
