File: hardware/vetrnik-power/vetrnik-power.kicad_pcb (KiCad board)
At the start: 2 copper layers, 124.5 x 99.1 mm, 138 parts, among them J1 12V IN, J10 AC1, J11 AC2, J12 G #Q3, J13 G #Q4, J14 AC frequency sense, J15 AVR-ISP-6, J16 ACS712_2, J17 ACS712, J2 ~SHORT, J3 UART, J4 ENABLE, J5 RELAYS, J6 DC IN, J7 PE, J8 G #Q1, J9 G #Q2, M1 12V / 0,9A max, Q1 BCP56-16, Q10 BC846, Q2 BC847, Q3 BC846, Q4 BC846, Q5 BC846, Q6 BC846, Q7 BC846, Q8 BC846, Q9 BC847, SW1 AVR RESET, U1 LTV-817, U10 LTV-817, U11 L78L05_TO92, U12 ATmega8-16PU, U2 LTV-817, U3 H11L1, U4 H11L1, U5 LTV-817, U6 LTV-847, U7 LM393, U8 IR2104, U9 IR2104, Y1 16MHz

Commit message: Migrate KiCAD projects to KiCAD 7.0
Parts:
- J2: value ~SHORT -> ~{SHORT}
Connections:
- net /AVR MCU/~ENABLE renamed /AVR MCU/~{ENABLE}
- net /AVR MCU/~RST renamed /AVR MCU/~{RST}
- net /AVR MCU/~SD renamed /AVR MCU/~{SD}
- net /AVR MCU/~SHORT renamed /AVR MCU/~{SHORT}
- net /H-bridge/~OVP renamed /H-bridge/~{OVP}
Other:
- net class Default removed

Commit message: [hardware] Clean up vetrnik-power schematic
Other:
- board text added: "This is the layout for the first prototype, which was later modified to connect to vetrnik-H-bridge. A redesign is needed if a new board is to be made."
