File: hardware/vetrnik-current-sensor-opamp/vetrnik-current-sensor-opamp.kicad_pcb (KiCad board)
At the start: 2 copper layers, 58.4 x 24.1 mm, 25 parts, among them J1 Conn_01x03, J2 Conn_Coaxial, J3 Conn_01x03, SW1 DP-06, U1 LMV358

Commit message: Migrate KiCAD projects to KiCAD 7.0
Other:
- net class Default removed
