File: hardware/vetrnik-current-sensor-opamp/vetrnik-current-sensor-opamp.kicad_sch (KiCad schematic)
At the start: 25 parts, among them J1 Conn_01x03, J2 Conn_Coaxial, J3 Conn_01x03, SW1 DP-06, U1 LMV358

Commit message: [hardware] Clean up vetrnik-current-sensor-opamp
Parts:
- added C6: 22p, symbol Device:C
- J2: value Conn_Coaxial -> BNC; Label (none) -> oscilloscope
- J3: Label POWER BOARD -> TO VETRNIK-POWER
Connections:
- net at J3.2 (Pin_2), R7.1, R8.2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: now also C6.2
- net at R5.1, R7.2, U1.2 (-): now also C6.1
Other:
- note added: "SW1 pins 8,9 connected for layout reasons"
- note added: "WARNING: +5V is +5P; GND is GNDPWR and so is the BNC shield."
- note added: "mod: added C6 to prevent parasitic oscillations"
- note removed: "TODO there were parasitic oscillations, 22pF added in parallel with R7"
- note removed: "WARNING: +5V is +5P; GND is GNDPWR and so is the BNC shield"
- company: (none) -> Ondřej Sluka
- title: (none) -> vetrnik-current-sensor-opamp
