File: hardware/vetrnik-power-supply/vetrnik-power-supply.kicad_pcb (KiCad board)
At the start: 2 copper layers, 80 x 21.6 mm, 21 parts, among them J1 Conn_01x02, J2 Conn_01x04, J3 Conn_01x04, J4 Conn_01x04, U1 LM2575-3.3BT, U2 LM7805_TO220

Commit message: Migrate KiCAD projects to KiCAD 7.0
Other:
- net class Default removed
