File: hardware/vetrnik-power-supply/vetrnik-power-supply.kicad_sch (KiCad schematic)
At the start: 21 parts, among them J1 Conn_01x02, J2 Conn_01x04, J3 Conn_01x04, J4 Conn_01x04, U1 LM2575-3.3BT, U2 LM7805_TO220

Commit message: [hardware] Clean up vetrnik-power-supply
Other:
- title: (none) -> vetrnik-power-supply
