File: hardware/vetrnik-relays/vetrnik-relays.kicad_pcb (KiCad board)
At the start: 2 copper layers, 48.3 x 73.7 mm, 14 parts, among them J1 Conn_01x04, J2 Screw_Terminal_01x03, J3 Screw_Terminal_01x03, J4 Screw_Terminal_01x03, K1 LEG-12F, K2 LEG-12F, K3 LEG-12F

Commit message: Migrate KiCAD projects to KiCAD 7.0
Other:
- net class Default removed

Commit message: [hardware] Clean up vetrnik-relays
Parts:
- K1, K2, K3: value LEG-12F -> 899-1CH-F-C-12VDC
Connections:
- net Net-(J2-Pad1) renamed /REL1_NC
- net Net-(J2-Pad2) renamed /REL1_COM
- net Net-(J2-Pad3) renamed /REL1_NO
- net Net-(J3-Pad1) renamed /REL2_NC
- net Net-(J3-Pad2) renamed /REL2_COM
- net Net-(J3-Pad3) renamed /REL2_NO
- net Net-(J4-Pad1) renamed /REL3_NC
- net Net-(J4-Pad2) renamed /REL3_COM
- net Net-(J4-Pad3) renamed /REL3_NO
Other:
- board text added: "TODO: screw terminal 3D models placed backwards"
