File: hardware/vetrnik-relays/vetrnik-relays.kicad_sch (KiCad schematic)
At the start: 14 parts, among them J1 Conn_01x04, J2 Screw_Terminal_01x03, J3 Screw_Terminal_01x03, J4 Screw_Terminal_01x03, K1 LEG-12F, K2 LEG-12F, K3 LEG-12F

Commit message: [hardware] Clean up vetrnik-relays
Parts:
- J1: Label (none) -> TO VETRNIK-CONTROL
- K1, K2, K3: value LEG-12F -> 899-1CH-F-C-12VDC
Connections:
- net REL1_COM: now reaches J2.2 (Pin_2), K1.11
- net REL1_NC: now reaches J2.1 (Pin_1), K1.12
- net REL1_NO: now reaches J2.3 (Pin_3), K1.14
- net REL2_NC: now reaches J3.1 (Pin_1), K2.12
- net REL2_COM: now reaches J3.2 (Pin_2), K2.11
- net REL2_NO: now reaches J3.3 (Pin_3), K2.14
- net REL3_NC: now reaches J4.1 (Pin_1), K3.12
- net REL3_COM: now reaches J4.2 (Pin_2), K3.11
- net REL3_NO: now reaches J4.3 (Pin_3), K3.14
Other:
- title: (none) -> vetrnik-relays
- moved on the sheet: J1, J2, J3, J4
