File: hardware/vetrnik-wind-sensor/vetrnik-wind-sensor.kicad_sch (KiCad schematic)
At the start: 41 parts, among them J1 NS25-W4P, J2 NS25-W4P, J3 Conn_01x08, J4 MTJ-88GX1-FSD, U1 AM1D-1224SH30Z, U2 RYK-0505S/H, U3 H11L1S(TA), U4 H11L1S(TA), U5 H11L1S(TA), U6 THVD1400DR

Commit message: [hardware] Clean up vetrnik-wind-sensor
Parts:
- J1: Label (none) -> TO VETRNIK-CONTROL
Other:
- company: (none) -> Ondřej Sluka
- title: (none) -> vetrnik-wind-sensor
- moved on the sheet: J1
Changed lines of the file:
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@@
 	(generator_version "8.0")
 	(paper "A4")
+	(title_block
+		(title "vetrnik-wind-sensor")
+		(company "Ondřej Sluka")
+	)
 	(junction
 		(at 96.52 171.45)
@@
 	(wire
 		(pts
-			(xy 25.4 78.74) (xy 34.29 78.74)
+			(xy 43.18 77.47) (xy 52.07 77.47)
 		)
 		(stroke
@@
 	(wire
 		(pts
-			(xy 25.4 76.2) (xy 34.29 76.2)
+			(xy 43.18 74.93) (xy 52.07 74.93)
 		)
 		(stroke
@@
 	(wire
 		(pts
-			(xy 29.21 81.28) (xy 25.4 81.28)
+			(xy 46.99 80.01) (xy 43.18 80.01)
 		)
 		(stroke
@@
 	(wire
 		(pts
-			(xy 25.4 73.66) (xy 34.29 73.66)
+			(xy 43.18 72.39) (xy 52.07 72.39)
 		)
 		(stroke
@@
 	(wire
 		(pts
-			(xy 29.21 82.55) (xy 29.21 81.28)
+			(xy 46.99 81.28) (xy 46.99 80.01)
 		)
 		(stroke
@@
 	(text "Sensor current < 15mA (specified <= 0.3W)\n28V TVS -> up to 16% out-of-spec 24V allowed.\nDC-DC Vout accuracy is +-3% & 1.2% Vout / 1% Vin"
 		(exclude_from_sim no)
-		(at 78.994 164.084 0)
+		(at 51.308 164.846 0)
 		(effects
 			(font
 				(size 1.27 1.27)
 			)
+			(justify left)
 		)
 	)
@@
 	)
 	(label "DE"
-		(at 34.29 78.74 180)
+		(at 52.07 77.47 180)
 		(effects
 			(font
@@
 	)
 	(label "TX"
-		(at 34.29 76.2 180)
+		(at 52.07 74.93 180)
 		(effects
 			(font
@@
 	)
 	(label "RX"
-		(at 34.29 73.66 180)
+		(at 52.07 72.39 180)
 		(effects
 			(font
@@
 	(symbol
 		(lib_id "power:GND")
-		(at 29.21 82.55 0)
+		(at 46.99 81.28 0)
 		(unit 1)
 		(exclude_from_sim no)
@@
 		(fields_autoplaced yes)
 		(property "Reference" "#PWR03"
-			(at 29.21 88.9 0)
+			(at 46.99 87.63 0)
 			(effects
 				(font
@@
 		)
 		(property "Value" "GND"
-			(at 29.21 86.6831 0)
+			(at 46.99 85.4131 0)
 			(effects
 				(font
@@
 		)
 		(property "Footprint" ""
-			(at 29.21 82.55 0)
+			(at 46.99 81.28 0)
 			(effects
 				(font
@@
 		)
 		(property "Datasheet" ""
-			(at 29.21 82.55 0)
+			(at 46.99 81.28 0)
 			(effects
 				(font
@@
 		)
 		(property "Description" "Power symbol creates a global label with name \"GND\" , ground"
-			(at 29.21 82.55 0)
+			(at 46.99 81.28 0)
 			(effects
 				(font
@@
 	(symbol
 		(lib_id "inventree:NS25-W4P")
-		(at 20.32 76.2 0)
+		(at 38.1 74.93 0)
 		(unit 1)
 		(exclude_from_sim no)
@@
 		(dnp no)
 		(property "Reference" "J1"
-			(at 20.955 71.8637 0)
+			(at 37.3888 73.7757 0)
 			(effects
 				(font
 					(size 1.27 1.27)
 				)
+				(justify right)
 			)
 		)
 		(property "Value" "NS25-W4P"
-			(at 20.955 69.4394 0)
+			(at 37.3888 76.2 0)
 			(effects
 				(font
 					(size 1.27 1.27)
 				)
+				(justify right)
 			)
 		)
 		(property "Footprint" "Connector_Molex:Molex_KK-254_AE-6410-04A_1x04_P2.54mm_Vertical"
-			(at 20.32 76.2 0)
+			(at 38.1 74.93 0)
 			(effects
 				(font
@@
 		)
 		(property "Datasheet" "http://inventree.rpi.lab.lan/media/attachments/part/452/ns25-w2p.pdf"
-			(at 20.32 76.2 0)
+			(at 38.1 74.93 0)
 			(effects
 				(font
@@
 		)
 		(property "Description" "Connector: wire-board; socket; male; NS25; 2.54mm; PIN: 4; THT; 250V"
-			(at 20.32 76.2 0)
+			(at 38.1 74.93 0)
 			(effects
 				(font
@@
 		)
 		(property "Connector Type" "socket"
-			(at 20.32 76.2 0)
+			(at 38.1 74.93 0)
 			(effects
 				(font
@@
 		)
 		(property "InvenTree" "452"
-			(at 20.32 76.2 0)
+			(at 38.1 74.93 0)
 			(effects
 				(font
@@
 		)
 		(property "Mounting Type" "THT"
-			(at 20.32 76.2 0)
+			(at 38.1 74.93 0)
 			(effects
 				(font
@@
 		)
 		(property "Number of Contacts" "4"
-			(at 20.32 76.2 0)
+			(at 38.1 74.93 0)
 			(effects
 				(font
@@
 		)
 		(property "Number of Rows" "1x4"
-			(at 20.32 76.2 0)
+			(at 38.1 74.93 0)
 			(effects
 				(font
@@
 		)
 		(property "Part URL" "http://inventree.rpi.lab.lan/part/452/"
-			(at 20.32 76.2 0)
+			(at 38.1 74.93 0)
 			(effects
 				(font
@@
 		)
 		(property "Pitch" "2.54mm"
-			(at 20.32 76.2 0)
+			(at 38.1 74.93 0)
 			(effects
 				(font
@@
 		)
 		(property "Rated Current" "3A"
-			(at 20.32 76.2 0)
+			(at 38.1 74.93 0)
 			(effects
 				(font
@@
 		)
 		(property "Rated Voltage" "0.25kV"
-			(at 20.32 76.2 0)
+			(at 38.1 74.93 0)
 			(effects
 				(font
@@
 			)
 		)
+		(property "Label" "TO VETRNIK-CONTROL"
+			(at 37.3888 78.6243 0)
+			(effects
+				(font
+					(size 1.27 1.27)
+				)
+				(justify right)
+			)
+		)
