File: hardware/vetrnik-control/vetrnik-control.kicad_pcb (KiCad board)
At the start: 2 copper layers, 99.1 x 76.2 mm, 87 parts, among them J1 Conn_01x20_Male, J10 Conn_01x04, J11 Conn_01x03_Male, J12 Conn_02x04_Odd_Even, J13 Conn_02x04_Odd_Even, J14 Conn_02x04_Odd_Even, J15 Conn_01x04, J16 Conn_01x04, J17 Conn_01x04, J18 Conn_01x03, J19 Conn_01x04, J2 Conn_01x04, J20 Conn_01x04, J3 Conn_01x03, J4 Conn_02x04_Odd_Even, J5 Conn_02x04_Odd_Even, J6 Conn_02x04_Odd_Even, J7 Conn_01x20_Male, J8 Screw_Terminal_01x02, J9 Conn_01x03, Q1 BC857, Q2 BC847, Q3 BC847, Q4 BC847, Q5 BSS138, Q6 BSS138, Q7 BC847, Q8 BSS138, SW1 SW_Push, SW2 SW_Push, U1 LTV-817S, U2 YAAJ_WeAct_BlackPill_Part_Like, U3 MX25L8006EM1I-12G, U4 WIZ850io

Commit message: Migrate KiCAD projects to KiCAD 7.0
Other:
- net class Default removed

Commit message: [hardware] Clean up vetrnik-control
Other:
- board text added: "TODO this is the layout for the prototype, there have been several modifications since then. A redesign is needed if a new board is to be made."
